Commit message: replace mesh with box
Signed-off-by: Karsten Knese <karsten@openrobotics.org>

File: dummy_robot/dummy_robot_bringup/launch/single_rrbot.urdf (robot description, URDF)
Before this commit: robot single_rrbot, 6 links, 5 joints
Links:
- link single_rrbot_hokuyo_link: geometry collision box size=0.1 0.1 0.1; visual box size=0.1 0.1 0.1
